File: hw/OpenUPS_ups/12V_Buck.kicad_sch (KiCad schematic)
At the start: 11 parts

Commit message: More cleanups and stuff
Parts:
- gave numbers to parts that had none: 5
Changed lines of the file:
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@@
   (symbol (lib_id "Regulator_Switching:AP63200WU") (at 138.43 104.14 0) (unit 1)
     (in_bom yes) (on_board yes) (dnp no) (fields_autoplaced)
-    (property "Reference" "U?" (at 138.43 95.3602 0)
+    (property "Reference" "U201" (at 138.43 95.3602 0)
       (effects (font (size 1.27 1.27)))
     )
@@
       (project "OpenUPS_ups"
         (path "/f77faec3-eac4-47f3-a2de-ec4a039f4502/a63ff227-b011-4ab9-8dd7-be9c5c5497e5"
-          (reference "U?") (unit 1)
+          (reference "U201") (unit 1)
         )
       )
@@
   (symbol (lib_id "Device:R_Small") (at 113.03 116.84 180) (unit 1)
     (in_bom yes) (on_board yes) (dnp no)
-    (property "Reference" "R?" (at 115.57 116.84 90)
+    (property "Reference" "R202" (at 115.57 116.84 90)
       (effects (font (size 1.27 1.27)))
     )
@@
       (project "OpenUPS_ups"
         (path "/f77faec3-eac4-47f3-a2de-ec4a039f4502/a63ff227-b011-4ab9-8dd7-be9c5c5497e5"
-          (reference "R?") (unit 1)
+          (reference "R202") (unit 1)
         )
       )
@@
   (symbol (lib_id "power:GND") (at 113.03 120.65 0) (unit 1)
     (in_bom yes) (on_board yes) (dnp no)
-    (property "Reference" "#PWR?" (at 113.03 127 0)
+    (property "Reference" "#PWR0104" (at 113.03 127 0)
       (effects (font (size 1.27 1.27)) hide)
     )
@@
       (project "OpenUPS_ups"
         (path "/f77faec3-eac4-47f3-a2de-ec4a039f4502/a63ff227-b011-4ab9-8dd7-be9c5c5497e5"
-          (reference "#PWR?") (unit 1)
+          (reference "#PWR0104") (unit 1)
         )
       )
@@
   (symbol (lib_id "Device:L") (at 172.72 95.25 90) (unit 1)
     (in_bom yes) (on_board yes) (dnp no)
-    (property "Reference" "L?" (at 172.72 90.424 90)
+    (property "Reference" "L201" (at 172.72 90.424 90)
       (effects (font (size 1.27 1.27)))
     )
@@
       (project "OpenUPS_ups"
         (path "/f77faec3-eac4-47f3-a2de-ec4a039f4502/a63ff227-b011-4ab9-8dd7-be9c5c5497e5"
-          (reference "L?") (unit 1)
+          (reference "L201") (unit 1)
         )
       )
@@
   (symbol (lib_id "power:GND") (at 217.17 107.95 0) (unit 1)
     (in_bom yes) (on_board yes) (dnp no)
-    (property "Reference" "#PWR?" (at 217.17 114.3 0)
+    (property "Reference" "#PWR0105" (at 217.17 114.3 0)
       (effects (font (size 1.27 1.27)) hide)
     )
@@
       (project "OpenUPS_ups"
         (path "/f77faec3-eac4-47f3-a2de-ec4a039f4502/a63ff227-b011-4ab9-8dd7-be9c5c5497e5"
-          (reference "#PWR?") (unit 1)
+          (reference "#PWR0105") (unit 1)
         )
       )
@@
   (symbol (lib_id "Device:C") (at 217.17 101.6 0) (mirror y) (unit 1)
     (in_bom yes) (on_board yes) (dnp no)
-    (property "Reference" "C?" (at 218.44 99.06 0)
+    (property "Reference" "C201" (at 218.44 99.06 0)
       (effects (font (size 1.27 1.27)) (justify right))
     )
@@
       (project "OpenUPS_ups"
         (path "/f77faec3-eac4-47f3-a2de-ec4a039f4502/a63ff227-b011-4ab9-8dd7-be9c5c5497e5"
-          (reference "C?") (unit 1)
+          (reference "C201") (unit 1)
         )
       )
@@
   (symbol (lib_id "Device:R_Small") (at 113.03 106.68 180) (unit 1)
     (in_bom yes) (on_board yes) (dnp no)
-    (property "Reference" "R?" (at 115.57 106.68 90)
+    (property "Reference" "R201" (at 115.57 106.68 90)
       (effects (font (size 1.27 1.27)))
     )
@@
       (project "OpenUPS_ups"
         (path "/f77faec3-eac4-47f3-a2de-ec4a039f4502/a63ff227-b011-4ab9-8dd7-be9c5c5497e5"
-          (reference "R?") (unit 1)
+          (reference "R201") (unit 1)
         )
       )
