File: hw/OpenUPS_ups/leds.kicad_sch (KiCad schematic)
At the start: 10 parts

Commit message: Initial placement effort
Parts:
- renumbered D1206 to D1101, D1201 to D1102, D1202 to D1103, D1203 to D1104, D1204 to D1105
Changed lines of the file:
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@@
         )
         (path "/f77faec3-eac4-47f3-a2de-ec4a039f4502/b8aa7be4-778b-4031-b56b-78965635bae2"
-          (reference "#PWR01201") (unit 1)
+          (reference "#PWR01101") (unit 1)
         )
       )
@@
         )
         (path "/f77faec3-eac4-47f3-a2de-ec4a039f4502/b8aa7be4-778b-4031-b56b-78965635bae2"
-          (reference "#PWR01204") (unit 1)
+          (reference "#PWR01104") (unit 1)
         )
       )
@@
         )
         (path "/f77faec3-eac4-47f3-a2de-ec4a039f4502/b8aa7be4-778b-4031-b56b-78965635bae2"
-          (reference "#PWR01202") (unit 1)
+          (reference "#PWR01102") (unit 1)
         )
       )
@@
         )
         (path "/f77faec3-eac4-47f3-a2de-ec4a039f4502/b8aa7be4-778b-4031-b56b-78965635bae2"
-          (reference "R1201") (unit 1)
+          (reference "R1101") (unit 1)
         )
       )
@@
   (symbol (lib_id "Device:LED_Small") (at 102.87 43.18 180) (unit 1)
     (in_bom yes) (on_board yes) (dnp no)
-    (property "Reference" "D1201" (at 100.33 46.99 0)
+    (property "Reference" "D1102" (at 100.33 46.99 0)
       (effects (font (size 1.27 1.27)) (justify right))
     )
@@
       (project "OpenUPS_ups"
         (path "/f77faec3-eac4-47f3-a2de-ec4a039f4502/b8aa7be4-778b-4031-b56b-78965635bae2"
-          (reference "D1201") (unit 1)
+          (reference "D1102") (unit 1)
         )
       )
@@
         )
         (path "/f77faec3-eac4-47f3-a2de-ec4a039f4502/b8aa7be4-778b-4031-b56b-78965635bae2"
-          (reference "#PWR01205") (unit 1)
+          (reference "#PWR01105") (unit 1)
         )
       )
@@
         )
         (path "/f77faec3-eac4-47f3-a2de-ec4a039f4502/b8aa7be4-778b-4031-b56b-78965635bae2"
-          (reference "R1203") (unit 1)
+          (reference "R1103") (unit 1)
         )
       )
@@
         )
         (path "/f77faec3-eac4-47f3-a2de-ec4a039f4502/b8aa7be4-778b-4031-b56b-78965635bae2"
-          (reference "R1205") (unit 1)
+          (reference "R1105") (unit 1)
         )
       )
@@
         )
         (path "/f77faec3-eac4-47f3-a2de-ec4a039f4502/b8aa7be4-778b-4031-b56b-78965635bae2"
-          (reference "R1202") (unit 1)
+          (reference "R1102") (unit 1)
         )
       )
@@
   (symbol (lib_id "Device:LED_Small") (at 102.87 66.04 180) (unit 1)
     (in_bom yes) (on_board yes) (dnp no)
-    (property "Reference" "D1203" (at 100.33 69.85 0)
+    (property "Reference" "D1104" (at 100.33 69.85 0)
       (effects (font (size 1.27 1.27)) (justify right))
     )
@@
       (project "OpenUPS_ups"
         (path "/f77faec3-eac4-47f3-a2de-ec4a039f4502/b8aa7be4-778b-4031-b56b-78965635bae2"
-          (reference "D1203") (unit 1)
+          (reference "D1104") (unit 1)
         )
       )
@@
   (symbol (lib_id "Device:LED_Small") (at 102.87 31.75 180) (unit 1)
     (in_bom yes) (on_board yes) (dnp no)
-    (property "Reference" "D1206" (at 100.33 35.56 0)
+    (property "Reference" "D1101" (at 100.33 35.56 0)
       (effects (font (size 1.27 1.27)) (justify right))
     )
@@
       (project "OpenUPS_ups"
         (path "/f77faec3-eac4-47f3-a2de-ec4a039f4502/b8aa7be4-778b-4031-b56b-78965635bae2"
-          (reference "D1206") (unit 1)
+          (reference "D1101") (unit 1)
         )
       )
@@
         )
         (path "/f77faec3-eac4-47f3-a2de-ec4a039f4502/b8aa7be4-778b-4031-b56b-78965635bae2"
-          (reference "#PWR01203") (unit 1)
+          (reference "#PWR01103") (unit 1)
         )
       )
@@
   (symbol (lib_id "Device:LED_Small") (at 102.87 77.47 180) (unit 1)
     (in_bom yes) (on_board yes) (dnp no)
-    (property "Reference" "D1204" (at 100.33 81.28 0)
+    (property "Reference" "D1105" (at 100.33 81.28 0)
       (effects (font (size 1.27 1.27)) (justify right))
     )
@@
       (project "OpenUPS_ups"
         (path "/f77faec3-eac4-47f3-a2de-ec4a039f4502/b8aa7be4-778b-4031-b56b-78965635bae2"
-          (reference "D1204") (unit 1)
+          (reference "D1105") (unit 1)
         )
       )
@@
         )
         (path "/f77faec3-eac4-47f3-a2de-ec4a039f4502/b8aa7be4-778b-4031-b56b-78965635bae2"
-          (reference "R1204") (unit 1)
+          (reference "R1104") (unit 1)
         )
       )
@@
   (symbol (lib_id "Device:LED_Small") (at 102.87 54.61 180) (unit 1)
     (in_bom yes) (on_board yes) (dnp no)
-    (property "Reference" "D1202" (at 100.33 58.42 0)
+    (property "Reference" "D1103" (at 100.33 58.42 0)
       (effects (font (size 1.27 1.27)) (justify right))
     )
@@
       (project "OpenUPS_ups"
         (path "/f77faec3-eac4-47f3-a2de-ec4a039f4502/b8aa7be4-778b-4031-b56b-78965635bae2"
-          (reference "D1202") (unit 1)
-        )
-      )
+          (reference "D1103") (unit 1)
+        )
+      )
