File: hw/OpenUPS_ups/ext_i2c.kicad_sch (KiCad schematic)
At the start: 11 parts, among them J7 Qwiic, U1001 π220N31

Commit message: Initial placement effort
Parts:
- R715: footprint (none) -> Resistor_SMD:R_0603_1608Metric
- renumbered U1001 to U901
Changed lines of the file:
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@@
       (effects (font (size 1.27 1.27)))
     )
-    (property "Footprint" "" (at 121.92 74.93 0)
+    (property "Footprint" "Resistor_SMD:R_0603_1608Metric" (at 121.92 74.93 0)
       (effects (font (size 1.27 1.27)) hide)
     )
@@
         )
         (path "/f77faec3-eac4-47f3-a2de-ec4a039f4502/8df8d962-7936-4f05-9ed7-4d48f457f001"
-          (reference "R1004") (unit 1)
+          (reference "R904") (unit 1)
         )
       )
@@
       (project "OpenUPS_ups"
         (path "/f77faec3-eac4-47f3-a2de-ec4a039f4502/8df8d962-7936-4f05-9ed7-4d48f457f001"
-          (reference "J1002") (unit 1)
+          (reference "J902") (unit 1)
         )
       )
@@
         )
         (path "/f77faec3-eac4-47f3-a2de-ec4a039f4502/8df8d962-7936-4f05-9ed7-4d48f457f001"
-          (reference "R1007") (unit 1)
+          (reference "R901") (unit 1)
         )
       )
@@
         )
         (path "/f77faec3-eac4-47f3-a2de-ec4a039f4502/8df8d962-7936-4f05-9ed7-4d48f457f001"
-          (reference "#PWR01001") (unit 1)
+          (reference "#PWR0901") (unit 1)
         )
       )
@@
   (symbol (lib_id "OpenUPS_ups:PAI220N31") (at 121.92 45.72 0) (unit 1)
     (in_bom yes) (on_board yes) (dnp no) (fields_autoplaced)
-    (property "Reference" "U1001" (at 121.92 42.7101 0)
+    (property "Reference" "U901" (at 121.92 42.7101 0)
       (effects (font (size 1.27 1.27)))
     )
@@
       (project "OpenUPS_ups"
         (path "/f77faec3-eac4-47f3-a2de-ec4a039f4502/8df8d962-7936-4f05-9ed7-4d48f457f001"
-          (reference "U1001") (unit 1)
+          (reference "U901") (unit 1)
         )
       )
@@
       (effects (font (size 1.27 1.27)))
     )
-    (property "Footprint" "" (at 121.92 67.31 0)
+    (property "Footprint" "Resistor_SMD:R_0603_1608Metric" (at 121.92 67.31 0)
       (effects (font (size 1.27 1.27)) hide)
     )
@@
         )
         (path "/f77faec3-eac4-47f3-a2de-ec4a039f4502/8df8d962-7936-4f05-9ed7-4d48f457f001"
-          (reference "R1003") (unit 1)
+          (reference "R903") (unit 1)
         )
       )
@@
         )
         (path "/f77faec3-eac4-47f3-a2de-ec4a039f4502/8df8d962-7936-4f05-9ed7-4d48f457f001"
-          (reference "R1001") (unit 1)
+          (reference "R906") (unit 1)
         )
       )
@@
         )
         (path "/f77faec3-eac4-47f3-a2de-ec4a039f4502/8df8d962-7936-4f05-9ed7-4d48f457f001"
-          (reference "C1001") (unit 1)
+          (reference "C901") (unit 1)
         )
       )
@@
         )
         (path "/f77faec3-eac4-47f3-a2de-ec4a039f4502/8df8d962-7936-4f05-9ed7-4d48f457f001"
-          (reference "R1002") (unit 1)
+          (reference "R905") (unit 1)
         )
       )
@@
         )
         (path "/f77faec3-eac4-47f3-a2de-ec4a039f4502/8df8d962-7936-4f05-9ed7-4d48f457f001"
-          (reference "C1002") (unit 1)
+          (reference "C902") (unit 1)
         )
       )
@@
         )
         (path "/f77faec3-eac4-47f3-a2de-ec4a039f4502/8df8d962-7936-4f05-9ed7-4d48f457f001"
-          (reference "#PWR01002") (unit 1)
+          (reference "#PWR0902") (unit 1)
         )
       )
@@
         )
         (path "/f77faec3-eac4-47f3-a2de-ec4a039f4502/8df8d962-7936-4f05-9ed7-4d48f457f001"
-          (reference "R1008") (unit 1)
+          (reference "R902") (unit 1)
         )
       )
@@
       (project "OpenUPS_ups"
         (path "/f77faec3-eac4-47f3-a2de-ec4a039f4502/8df8d962-7936-4f05-9ed7-4d48f457f001"
-          (reference "J1001") (unit 1)
-        )
-      )
+          (reference "J901") (unit 1)
+        )
+      )

Commit message: PCB multitasking
Parts:
- removed R715 (x2): NM, Resistor_SMD:R_0603_1608Metric, symbol Device:R_Small
Other:
- note removed: "Overlapping with isolator chip In case no isolation is needed"
Changed lines of the file:
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@@
-    (stroke (width 0) (type default))
-  )
-  (wire (pts (xy 88.9 67.31) (xy 88.9 55.88))
     (stroke (width 0) (type default))
   )
@@
     (stroke (width 0) (type default))
   )
-  (wire (pts (xy 80.01 74.93) (xy 80.01 50.8))
-    (stroke (width 0) (type default))
-  )
   (wire (pts (xy 163.83 43.18) (xy 154.94 43.18))
     (stroke (width 0) (type default))
@@
     (stroke (width 0) (type default))
   )
-  (wire (pts (xy 124.46 74.93) (xy 163.83 74.93))
-    (stroke (width 0) (type default))
-  )
   (wire (pts (xy 80.01 44.45) (xy 80.01 43.18))
     (stroke (width 0) (type default))
@@
     (stroke (width 0) (type default))
   )
-  (wire (pts (xy 163.83 74.93) (xy 163.83 50.8))
-    (stroke (width 0) (type default))
-  )
   (wire (pts (xy 146.05 58.42) (xy 134.62 58.42))
     (stroke (width 0) (type default))
@@
     (stroke (width 0) (type default))
   )
-  (wire (pts (xy 119.38 74.93) (xy 80.01 74.93))
-    (stroke (width 0) (type default))
-  )
   (wire (pts (xy 74.93 55.88) (xy 88.9 55.88))
     (stroke (width 0) (type default))
@@
     (stroke (width 0) (type default))
   )
-  (wire (pts (xy 124.46 67.31) (xy 154.94 67.31))
-    (stroke (width 0) (type default))
-  )
   (wire (pts (xy 146.05 49.53) (xy 146.05 58.42))
     (stroke (width 0) (type default))
@@
     (stroke (width 0) (type default))
   )
-  (wire (pts (xy 154.94 67.31) (xy 154.94 55.88))
-    (stroke (width 0) (type default))
-  )
   (wire (pts (xy 74.93 58.42) (xy 97.79 58.42))
     (stroke (width 0) (type default))
@@
     (stroke (width 0) (type default))
   )
-  (wire (pts (xy 119.38 67.31) (xy 88.9 67.31))
-    (stroke (width 0) (type default))
-  )
   (wire (pts (xy 168.91 39.37) (xy 168.91 43.18))
     (stroke (width 0) (type default))
@@
   (wire (pts (xy 88.9 49.53) (xy 88.9 55.88))
     (stroke (width 0) (type default))
-  )
-  (rectangle (start 115.57 62.23) (end 128.27 80.01)
-    (stroke (width 0) (type dash))
-    (fill (type none))
-  )
-  (text "Overlapping with isolator chip\nIn case no isolation is needed"
-    (at 107.95 85.09 0)
-    (effects (font (size 1.27 1.27)) (justify left bottom))
   )
   (label "XI2C_GND" (at 40.64 72.39 0) (fields_autoplaced)
@@
   (hierarchical_label "Ext_SDA" (shape bidirectional) (at 168.91 50.8 0) (fields_autoplaced)
     (effects (font (size 1.27 1.27)) (justify left))
-  )
-  (symbol (lib_id "Device:R_Small") (at 121.92 74.93 90) (unit 1)
-    (in_bom yes) (on_board yes) (dnp no)
-    (property "Reference" "R715" (at 121.92 72.39 90)
-      (effects (font (size 1.27 1.27)))
-    )
-    (property "Value" "NM" (at 121.92 77.47 90)
-      (effects (font (size 1.27 1.27)))
-    )
-    (property "Footprint" "Resistor_SMD:R_0603_1608Metric" (at 121.92 74.93 0)
-      (effects (font (size 1.27 1.27)) hide)
-    )
-    (property "Datasheet" "~" (at 121.92 74.93 0)
-      (effects (font (size 1.27 1.27)) hide)
-    )
-    (pin "1")
-    (pin "2")
-    (instances
-      (project "OpenUPS_ups"
-        (path "/f77faec3-eac4-47f3-a2de-ec4a039f4502/09fcd86a-cc7e-4bce-97cb-42a94055ba63"
-          (reference "R715") (unit 1)
-        )
-        (path "/f77faec3-eac4-47f3-a2de-ec4a039f4502/dfbaaed0-e564-4e21-900d-d5a65c0f1694"
-          (reference "R413") (unit 1)
-        )
-        (path "/f77faec3-eac4-47f3-a2de-ec4a039f4502/0bd99307-a15c-41e8-997b-077d576f806c"
-          (reference "R509") (unit 1)
-        )
-        (path "/f77faec3-eac4-47f3-a2de-ec4a039f4502/8df8d962-7936-4f05-9ed7-4d48f457f001"
-          (reference "R904") (unit 1)
-        )
-      )
-    )
   )
   (symbol (lib_id "Connector_Generic_MountingPin:Conn_01x04_MountingPin") (at 29.21 74.93 0) (mirror y) (unit 1)
@@
         )
       )
-    )
-  )
-  (symbol (lib_id "Device:R_Small") (at 121.92 67.31 90) (unit 1)
-    (in_bom yes) (on_board yes) (dnp no)
-    (property "Reference" "R715" (at 121.92 64.77 90)
-      (effects (font (size 1.27 1.27)))
-    )
-    (property "Value" "NM" (at 121.92 69.85 90)
-      (effects (font (size 1.27 1.27)))
-    )
-    (property "Footprint" "Resistor_SMD:R_0603_1608Metric" (at 121.92 67.31 0)
-      (effects (font (size 1.27 1.27)) hide)
-    )
-    (property "Datasheet" "~" (at 121.92 67.31 0)
-      (effects (font (size 1.27 1.27)) hide)
-    )
-    (pin "1")
-    (pin "2")
-    (instances
-      (project "OpenUPS_ups"
-        (path "/f77faec3-eac4-47f3-a2de-ec4a039f4502/09fcd86a-cc7e-4bce-97cb-42a94055ba63"
-          (reference "R715") (unit 1)
-        )
-        (path "/f77faec3-eac4-47f3-a2de-ec4a039f4502/dfbaaed0-e564-4e21-900d-d5a65c0f1694"
-          (reference "R413") (unit 1)
-        )
-        (path "/f77faec3-eac4-47f3-a2de-ec4a039f4502/0bd99307-a15c-41e8-997b-077d576f806c"
-          (reference "R509") (unit 1)
-        )
-        (path "/f77faec3-eac4-47f3-a2de-ec4a039f4502/8df8d962-7936-4f05-9ed7-4d48f457f001"
-          (reference "R903") (unit 1)
-        )
-      )
